File: kicad_source/CANFDZeroHAT.sch (KiCad schematic (older format))
At the start: 31 parts, among them CN1 RASPI-IO, CN2 691322310004, CN3 GH_SM04B-GHS-TB, CN4 GH_SM04B-GHS-TB, SW1 JS202011JCQN, U1 MCP2518FD, U2 TCAN332GDR, Y1 RH100-20.000-20-3030-TR

Commit message: updated layout
Parts:
- D2, D3, D4: footprint (none) -> LEDs:LED_0603
Changed lines of the file:
@@
 F 0 "D2" H 6200 3095 50  0000 C CNN
 F 1 "150060GS75000" H 6200 3186 50  0000 C CNN
-F 2 "" V 6200 3300 50  0000 C CNN
+F 2 "LEDs:LED_0603" V 6200 3300 50  0001 C CNN
 F 3 "" V 6200 3300 50  0000 C CNN
 	1    6200 3300
@@
 F 0 "D3" H 6200 3445 50  0000 C CNN
 F 1 "150060RS75000" H 6200 3536 50  0000 C CNN
-F 2 "" V 6200 3650 50  0000 C CNN
+F 2 "LEDs:LED_0603" V 6200 3650 50  0001 C CNN
 F 3 "" V 6200 3650 50  0000 C CNN
 	1    6200 3650
@@
 F 0 "D4" H 6200 3795 50  0000 C CNN
 F 1 "150060YS75000" H 6200 3886 50  0000 C CNN
-F 2 "" V 6200 4000 50  0000 C CNN
+F 2 "LEDs:LED_0603" V 6200 4000 50  0001 C CNN
 F 3 "" V 6200 4000 50  0000 C CNN
 	1    6200 4000

Commit message: corrected footprint of CAN transceiver
Parts:
- U2: footprint SOIC:SOIJ-8_5.3x5.3mm_Pitch1.27mm -> SOIC:SOIC-8_3.9x4.9mm_Pitch1.27mm
Changed lines of the file:
@@
 F 0 "U2" H 4775 2887 60  0000 C CNN
 F 1 "TCAN332GDR" H 4775 2781 60  0000 C CNN
-F 2 "SOIC:SOIJ-8_5.3x5.3mm_Pitch1.27mm" H 5100 1950 60  0001 C CNN
+F 2 "SOIC:SOIC-8_3.9x4.9mm_Pitch1.27mm" H 5100 1950 60  0001 C CNN
 F 3 "" H 4250 2150 60  0000 C CNN
 	1    4250 2000
